Commit message: Added new features

File: jetbot_orgon_description/urdf/jetbot.urdf.xacro (robot description, xacro)
@@ -9,5 +9,5 @@
     <material name="grey"> <color rgba="0.5 0.5 0.5 1"/> </material>
     <!-- Odom link (корень без инерции и коллизии) -->
-    <link name="odom"/>
+    <!-- <link name="odom"/> -->
     <!-- Корпус джетбота (с инерцией и коллизией) -->
     <link name="base_link">
@@ -31,11 +31,11 @@
         </inertial>
     </link>
-    <joint name="base_link_joint" type="fixed">
+    <!-- <joint name="base_link_joint" type="fixed">
         <parent link="odom"/>
         <child link="base_link"/>
         <origin xyz="0 0 0" rpy="0 0 0"/>
-    </joint>
+    </joint> -->
     <!-- RP-Lidar (с коллизией и инерцией) -->
-    <link name="lidar">
+    <link name="lidar_link">
         <visual>
             <geometry>
@@ -59,9 +59,9 @@
     <joint name="base_link_lidar_joint" type="fixed">
         <parent link="base_link"/>
-        <child link="lidar"/>
-        <origin xyz="0.11491 0 -0.0239" rpy="0 0 0"/>
+        <child link="lidar_link"/>
+        <origin xyz="0.11491 0 -0.0239" rpy="0 0 2.3562"/>
     </joint>
     <!-- Left wheel (с коллизией и инерцией) -->
-    <link name="left_wheel">
+    <link name="left_wheel_link">
         <visual>
             <geometry>
@@ -85,10 +85,10 @@
     <joint name="base_link_left_wheel_joint" type="continuous">
         <parent link="base_link"/>
-        <child link="left_wheel"/>
+        <child link="left_wheel_link"/>
         <origin xyz="0.03004 0.08107 -0.00937" rpy="0 0 0"/>
         <axis xyz="0 1 0"/>
     </joint>
     <!-- Right wheel (с коллизией и инерцией) -->
-    <link name="right_wheel">
+    <link name="right_wheel_link">
         <visual>
             <geometry>
@@ -112,10 +112,10 @@
     <joint name="base_link_right_wheel_joint" type="continuous">
         <parent link="base_link"/>
-        <child link="right_wheel"/>
+        <child link="right_wheel_link"/>
         <origin xyz="0.03004 -0.08107 -0.00937" rpy="0 0 0"/>
         <axis xyz="0 1 0"/>
     </joint>
     <!-- Платформа манипулятора -->
-    <link name="manipulator_platform">
+    <link name="manipulator_platform_link">
         <visual>
             <geometry>
@@ -139,5 +139,5 @@
     <joint name="base_link_manipulator_platform_joint" type="fixed">
         <parent link="base_link"/>
-        <child link="manipulator_platform"/>
+        <child link="manipulator_platform_link"/>
         <origin xyz="0.07491 0 0.0239" rpy="0 0 0"/>
     </joint>
@@ -165,10 +165,10 @@
     </link>
     <joint name="manipulator_platform_manipulator_base_link_joint" type="fixed">
-        <parent link="manipulator_platform"/>
+        <parent link="manipulator_platform_link"/>
         <child link="manipulator_base_link"/>
         <origin xyz="0.04302 0.01263 0.02805" rpy="0 0 0"/>
     </joint>
     <!-- Шарнир на базе -->
-    <link name="base_joint_visual">
+    <link name="base_joint_visual_link">
         <visual>
             <geometry>
@@ -181,5 +181,5 @@
     <joint name="manipulator_base_joint_visual_joint" type="fixed">
         <parent link="manipulator_base_link"/>
-        <child link="base_joint_visual"/>
+        <child link="base_joint_visual_link"/>
         <origin xyz="0.0101 -0.015 0.00655" rpy="0 0 0"/>
     </joint>
@@ -384,5 +384,5 @@
     <!-- =============================================================== Манипулятор =============================================================== -->
     <!-- Мозги (с инерцией и коллизией) -->
-    <link name="sandwich">
+    <link name="sandwich_link">
         <visual>
             <geometry>
@@ -406,9 +406,9 @@
     <joint name="base_link_sandwich_joint" type="fixed">
         <parent link="base_link"/>
-        <child link="sandwich"/>
+        <child link="sandwich_link"/>
         <origin xyz="0.0075 -0.004 0.024" rpy="0 0 0"/>
     </joint>
     <!-- Левая антенна (с коллизией и инерцией) -->
-    <link name="left_antenn">
+    <link name="left_antenn_link">
         <visual>
             <geometry>
@@ -432,9 +432,9 @@
     <joint name="base_link_left_antenn_joint" type="fixed">
         <parent link="base_link"/>
-        <child link="left_antenn"/>
+        <child link="left_antenn_link"/>
         <origin xyz="-0.075 0.045 0.024" rpy="0 0 0"/>
     </joint>
     <!-- Правая антенна (с коллизией и инерцией) -->
-    <link name="right_antenn">
+    <link name="right_antenn_link">
         <visual>
             <geometry>
@@ -458,5 +458,5 @@
     <joint name="base_link_right_antenn_joint" type="fixed">
         <parent link="base_link"/>
-        <child link="right_antenn"/>
+        <child link="right_antenn_link"/>
         <origin xyz="-0.075 -0.045 0.024" rpy="0 0 0"/>
     </joint>

Commit message: urdf fixed

File: jetbot_orgon_description/urdf/jetbot.urdf.xacro (robot description, xacro)
@@ -8,6 +8,6 @@
     <material name="silver"> <color rgba="0.75 0.75 0.75 1"/> </material>
     <material name="grey"> <color rgba="0.5 0.5 0.5 1"/> </material>
-    <!-- Odom link (корень без инерции и коллизии) -->
-    <!-- <link name="odom"/> -->
+    <!-- Odom link (корень без инерции и коллизии)
+    <link name="odom"/> -->
     <!-- Корпус джетбота (с инерцией и коллизией) -->
     <link name="base_link">
@@ -37,5 +37,5 @@
     </joint> -->
     <!-- RP-Lidar (с коллизией и инерцией) -->
-    <link name="lidar_link">
+    <link name="lidar">
         <visual>
             <geometry>
@@ -59,9 +59,9 @@
     <joint name="base_link_lidar_joint" type="fixed">
         <parent link="base_link"/>
-        <child link="lidar_link"/>
+        <child link="lidar"/>
         <origin xyz="0.11491 0 -0.0239" rpy="0 0 2.3562"/>
     </joint>
     <!-- Left wheel (с коллизией и инерцией) -->
-    <link name="left_wheel_link">
+    <link name="left_wheel">
         <visual>
             <geometry>
@@ -85,10 +85,10 @@
     <joint name="base_link_left_wheel_joint" type="continuous">
         <parent link="base_link"/>
-        <child link="left_wheel_link"/>
+        <child link="left_wheel"/>
         <origin xyz="0.03004 0.08107 -0.00937" rpy="0 0 0"/>
         <axis xyz="0 1 0"/>
     </joint>
     <!-- Right wheel (с коллизией и инерцией) -->
-    <link name="right_wheel_link">
+    <link name="right_wheel">
         <visual>
             <geometry>
@@ -112,10 +112,10 @@
     <joint name="base_link_right_wheel_joint" type="continuous">
         <parent link="base_link"/>
-        <child link="right_wheel_link"/>
+        <child link="right_wheel"/>
         <origin xyz="0.03004 -0.08107 -0.00937" rpy="0 0 0"/>
         <axis xyz="0 1 0"/>
     </joint>
     <!-- Платформа манипулятора -->
-    <link name="manipulator_platform_link">
+    <link name="manipulator_platform">
         <visual>
             <geometry>
@@ -139,5 +139,5 @@
     <joint name="base_link_manipulator_platform_joint" type="fixed">
         <parent link="base_link"/>
-        <child link="manipulator_platform_link"/>
+        <child link="manipulator_platform"/>
         <origin xyz="0.07491 0 0.0239" rpy="0 0 0"/>
     </joint>
@@ -165,10 +165,10 @@
     </link>
     <joint name="manipulator_platform_manipulator_base_link_joint" type="fixed">
-        <parent link="manipulator_platform_link"/>
+        <parent link="manipulator_platform"/>
         <child link="manipulator_base_link"/>
-        <origin xyz="0.04302 0.01263 0.02805" rpy="0 0 0"/>
+        <origin xyz="0.04302 -0.0137 0.02805" rpy="0 0 0"/>
     </joint>
     <!-- Шарнир на базе -->
-    <link name="base_joint_visual_link">
+    <link name="base_hinge">
         <visual>
             <geometry>
@@ -179,7 +179,7 @@
         </visual>
     </link>
-    <joint name="manipulator_base_joint_visual_joint" type="fixed">
+    <joint name="manipulator_base_hinge_joint" type="fixed">
         <parent link="manipulator_base_link"/>
-        <child link="base_joint_visual_link"/>
+        <child link="base_hinge"/>
         <origin xyz="0.0101 -0.015 0.00655" rpy="0 0 0"/>
     </joint>
@@ -213,5 +213,5 @@
     </joint>
     <!-- Шарнир между первым и вторым звеном -->
-    <link name="first_joint_visual">
+    <link name="first_link_hinge">
         <visual>
             <geometry>
@@ -222,7 +222,7 @@
         </visual>
     </link>
-    <joint name="first_joint_visual_joint" type="fixed">
+    <joint name="first_link_first_link_hinge_joint" type="fixed">
         <parent link="first_link"/>
-        <child link="first_joint_visual"/>
+        <child link="first_link_hinge"/>
         <origin xyz="0.0634 0.0051 0" rpy="0 0 0"/>
     </joint>
@@ -256,5 +256,5 @@
     </joint>
     <!-- Крепление платформы -->
-    <link name="second_joint_visual">
+    <link name="second_link_fastening">
         <visual>
             <geometry>
@@ -265,7 +265,7 @@
         </visual>
     </link>
-    <joint name="second_joint_visual_joint" type="fixed">
+    <joint name="second_link_second_link_fastening_joint" type="fixed">
         <parent link="second_link"/>
-        <child link="second_joint_visual"/>
+        <child link="second_link_fastening"/>
         <origin xyz="0.0482 0.00825 -0.0035" rpy="0 0 0"/>
     </joint>
@@ -297,5 +297,5 @@
     </joint>
     <!--  Шарнир левого хвата -->
-    <link name="left_finger_joint_visual">
+    <link name="left_finger_hinge">
         <visual>
             <geometry>
@@ -306,7 +306,7 @@
         </visual>
     </link>
-    <joint name="left_finger_joint_visual_joint" type="fixed">
+    <joint name="left_finger_left_finger_hinge_joint" type="fixed">
         <parent link="second_link_platform"/>
-        <child link="left_finger_joint_visual"/>
+        <child link="left_finger_hinge"/>
         <origin xyz="0.023 0.0092 -0.006" rpy="0 0 0"/>
     </joint>
@@ -340,5 +340,5 @@
     </joint>
     <!-- Шарнир правого хвата -->
-    <link name="right_finger_joint_visual">
+    <link name="right_finger_hinge">
         <visual>
             <geometry>
@@ -349,7 +349,7 @@
         </visual>
     </link>
-    <joint name="right_finger_joint_visual_joint" type="fixed">
+    <joint name="right_finger_right_finger_hinge_joint" type="fixed">
         <parent link="second_link_platform"/>
-        <child link="right_finger_joint_visual"/>
+        <child link="right_finger_hinge"/>
         <origin xyz="0.023 -0.0092 -0.006" rpy="0 0 0"/>
     </joint>
@@ -384,5 +384,5 @@
     <!-- =============================================================== Манипулятор =============================================================== -->
     <!-- Мозги (с инерцией и коллизией) -->
-    <link name="sandwich_link">
+    <link name="sandwich">
         <visual>
             <geometry>
@@ -406,9 +406,9 @@
     <joint name="base_link_sandwich_joint" type="fixed">
         <parent link="base_link"/>
-        <child link="sandwich_link"/>
+        <child link="sandwich"/>
         <origin xyz="0.0075 -0.004 0.024" rpy="0 0 0"/>
     </joint>
     <!-- Левая антенна (с коллизией и инерцией) -->
-    <link name="left_antenn_link">
+    <link name="left_antenn">
         <visual>
             <geometry>
@@ -432,9 +432,9 @@
     <joint name="base_link_left_antenn_joint" type="fixed">
         <parent link="base_link"/>
-        <child link="left_antenn_link"/>
+        <child link="left_antenn"/>
         <origin xyz="-0.075 0.045 0.024" rpy="0 0 0"/>
     </joint>
     <!-- Правая антенна (с коллизией и инерцией) -->
-    <link name="right_antenn_link">
+    <link name="right_antenn">
         <visual>
             <geometry>
@@ -458,5 +458,5 @@
     <joint name="base_link_right_antenn_joint" type="fixed">
         <parent link="base_link"/>
-        <child link="right_antenn_link"/>
+        <child link="right_antenn"/>
         <origin xyz="-0.075 -0.045 0.024" rpy="0 0 0"/>
     </joint>

Commit message: visual Pavel

File: jetbot_orgon_description/urdf/jetbot.urdf.xacro (robot description, xacro)
@@ -37,5 +37,5 @@
     </joint> -->
     <!-- RP-Lidar (с коллизией и инерцией) -->
-    <link name="lidar">
+    <link name="lidar_link">
         <visual>
             <geometry>
@@ -59,5 +59,5 @@
     <joint name="base_link_lidar_joint" type="fixed">
         <parent link="base_link"/>
-        <child link="lidar"/>
+        <child link="lidar_link"/>
         <origin xyz="0.11491 0 -0.0239" rpy="0 0 2.3562"/>
     </joint>
